File: power_manager_ports.sch (EAGLE design)
At the start: 0 parts

Commit message: added basics ports
Parts:
- added X1: (no value), con-wago-500:W239-302
- added X3: C-GRID-07-70543, con-molex:C-GRID-07-70543
- added X4: C-GRID-05-70543, con-molex:C-GRID-05-70543
- added X5: C-GRID-06-70543, con-molex:C-GRID-06-70543
Connections:
- new net 24V: X1-1.KL
- new net 3.3V: X3-7.S, X4-5.S, X5-6.S
- new net 5V: X3-6.S, X4-4.S, X5-5.S
- new net CAN_0: X5-1.S
- new net CAN_1: X5-2.S
- new net CLK: X3-3.S
- new net GND: X1-2.KL, X3-5.S, X4-3.S, X5-3.S, X5-4.S
- new net MISO: X3-2.S
- new net MOSI: X3-1.S
- new net SCL: X4-2.S
- new net SDA: X4-1.S
- new net SS: X3-4.S
